File: hardware/hardfuzz_v1/board.kicad_sch (KiCad schematic)
At the start: 68 parts, among them J1 USB-C, J2 Qwiic, J3 BUS, J4 SPI/UART, J5 CAN, SW1 PROG, U1 XC7A35T-CSG324, U10 TXS0108EPW, U2 FT2232HQ, U3 MX25L3233F, U6 TLV62566, U7 TLV62566, U8 AP2112K-1.8, U9 SN65HVD230, Y1 12MHz, Y2 12MHz

Commit message: hardware(kigen): hierarchical schematic — one readable page per subsystem
Reorganise the flat board into a hierarchical KiCad project: root board.kicad_sch
instantiates five sub-sheets (FPGA/Power/CAN/Level-Shift/USB), each its own legible
page. kigen gains global-label + hierarchical-instance-path support; build_board
auto-detects cross-sheet nets (24) and emits them as global labels, keeping block-
internal nets local. Verified: root loads and renders 6 pages, cross-sheet netlist
connects (SPI/JTAG/flash/CAN/VREF span sheets), 0 collisions, and the kicad-happy
skill parses all 6 sheets at HIGH trust.

Co-Authored-By: Claude Opus 4.8 <noreply@anthropic.com>
Parts:
- removed C1, C2, C40, C47: 10uF, Capacitor_SMD:C_0402_1005Metric, symbol Device:C
- removed C20, C30, C31, C41, C43, C44, C48, C50: 100nF, Capacitor_SMD:C_0402_1005Metric, symbol Device:C
- removed C21: 4.7nF, Capacitor_SMD:C_0402_1005Metric, symbol Device:C
- removed C3, C4, C5, C6: 22uF, Capacitor_SMD:C_0402_1005Metric, symbol Device:C
- removed C32, C7, C8: 1uF, Capacitor_SMD:C_0402_1005Metric, symbol Device:C
- removed C42, C51, C52, C53: 4.7uF, Capacitor_SMD:C_0402_1005Metric, symbol Device:C
- removed C45, C46: 18pF, Capacitor_SMD:C_0402_1005Metric, symbol Device:C
- removed D20: SMAJ5.0A, Diode_SMD:D_SOD-923, symbol Device:D_TVS
- removed D30: USBLC6-2SC6, Package_TO_SOT_SMD:SOT-23-6, symbol Power_Protection:USBLC6-2SC6
- removed D31: SMAJ5.0A, Diode_SMD:D_SMA, symbol Device:D_TVS
- removed D40: DONE, LED_SMD:LED_0603_1608Metric, symbol Device:LED
- removed J1: USB-C, Connector_USB:USB_C_Receptacle_GCT_USB4085, symbol Connector:USB_C_Receptacle
- removed J2: Qwiic, Connector_JST:JST_SH_SM04B-SRSS-TB_1x04-1MP_P1.00mm_Horizontal, symbol Connector_Generic:Conn_01x04
- removed J3: BUS, Connector_PinHeader_2.54mm:PinHeader_2x10_P2.54mm_Vertical, symbol Connector_Generic:Conn_02x10_Odd_Even
- removed J4: SPI/UART, Connector_PinHeader_2.54mm:PinHeader_2x05_P2.54mm_Vertical, symbol Connector_Generic:Conn_02x05_Odd_Even
- removed J5: CAN, TerminalBlock_Phoenix:TerminalBlock_Phoenix_MPT-0,5-3-2.54_1x03, symbol Connector:Screw_Terminal_01x03
- removed L1: 2.2uH, Inductor_SMD:L_0805_2012Metric, symbol Device:L
- removed L2: 1.5uH, Inductor_SMD:L_0805_2012Metric, symbol Device:L
- removed R1: 412k, Resistor_SMD:R_0402_1005Metric, symbol Device:R
- removed R2: 91k, Resistor_SMD:R_0402_1005Metric, symbol Device:R
- removed R20, R40, R43: 10k, Resistor_SMD:R_0402_1005Metric, symbol Device:R
- removed R21, R22: 60R, Resistor_SMD:R_0402_1005Metric, symbol Device:R
- removed R3: 133k, Resistor_SMD:R_0402_1005Metric, symbol Device:R
- removed R30, R33, R34: 100k, Resistor_SMD:R_0402_1005Metric, symbol Device:R
- removed R31, R32, R50, R51: 4.7k, Resistor_SMD:R_0402_1005Metric, symbol Device:R
- removed R4: 200k, Resistor_SMD:R_0402_1005Metric, symbol Device:R
- removed R41, R42: 5.1k, Resistor_SMD:R_0402_1005Metric, symbol Device:R
- removed R52: 3.3k, Resistor_SMD:R_0402_1005Metric, symbol Device:R
- removed R53: 330, Resistor_SMD:R_0402_1005Metric, symbol Device:R
- removed SW1: PROG, Button_Switch_SMD:SW_SPST_CK_RS282G05A3, symbol Switch:SW_Push
- removed U1: XC7A35T-CSG324, Package_BGA:Xilinx_CSG324, symbol FPGA_Xilinx_Artix7:XC7A35T-CSG324
- removed U10: TXS0108EPW, symbol Logic_LevelTranslator:TXS0108EPW
- removed U2: FT2232HQ, symbol Interface_USB:FT2232HQ
- removed U3: MX25L3233F, Package_SO:SOIC-8_5.23x5.23mm_P1.27mm, symbol Memory_Flash:MX25L3233FM
- removed U6, U7: TLV62566, symbol Regulator_Switching:TLV62566DBVx
- removed U8: AP2112K-1.8, symbol Regulator_Linear:AP2112K-1.8
- removed U9: SN65HVD230, symbol Interface_CAN_LIN:SN65HVD230
- removed Y1: 12MHz, Oscillator:Oscillator_SMD_Abracon_ASE-4Pin_3.2x2.5mm, symbol Oscillator:ASE-xxxMHz
- removed Y2: 12MHz, Crystal:Crystal_SMD_3225-4Pin_3.2x2.5mm, symbol Device:Crystal_GND24
Other:
- added sheet CAN (can.kicad_sch)
- added sheet FPGA (fpga.kicad_sch)
- added sheet Level Shift (levelshift.kicad_sch)
- added sheet Power (power.kicad_sch)
- added sheet USB (usb.kicad_sch)
