File: hardware/hardfuzz_v1/fpga.kicad_sch (KiCad schematic)
At the start: 12 parts, among them SW1 PROG, U1 XC7A35T-CSG324, Y1 12MHz

Commit message: hardware(kigen): review cleanup — NC flags, MPNs, PG/flag fixes, FPGA on A1
Address kicad-happy skill + ERC findings on the hierarchical board:
- no-connect flags on all intentional spare pins (unconnected 238 -> 0)
- MPNs on 16 ICs/connectors; grid-snapped endpoints
- fix buck PG mis-map (was tied to VIN) and drop double-driver PWR_FLAGs
- rename FT core rail VDDCORE_FT so PP-001 reads it as an internal rail (info)
- FPGA sub-sheet on A1 so all 5 units fit on the page
kigen gains no_connect + MPN emission. Skill review now: 1 error (SS-001
sourcing gate, needs passive MPNs) + benign info; netlist connectivity intact.

Co-Authored-By: Claude Opus 4.8 <noreply@anthropic.com>
Parts:
- U1: MPN (none) -> XC7A35T-1CSG324C
- Y1: MPN (none) -> ASE-12.000MHZ-LC-T
Connections:
- no-connect marks 0 -> 196
