File: hardware/hardfuzz_v1/levelshift.kicad_sch (KiCad schematic)
At the start: 13 parts, among them J2 Qwiic, J3 BUS, J4 SPI/UART, U10 TXS0108EPW

Commit message: hardware(kigen): review cleanup — NC flags, MPNs, PG/flag fixes, FPGA on A1
Address kicad-happy skill + ERC findings on the hierarchical board:
- no-connect flags on all intentional spare pins (unconnected 238 -> 0)
- MPNs on 16 ICs/connectors; grid-snapped endpoints
- fix buck PG mis-map (was tied to VIN) and drop double-driver PWR_FLAGs
- rename FT core rail VDDCORE_FT so PP-001 reads it as an internal rail (info)
- FPGA sub-sheet on A1 so all 5 units fit on the page
kigen gains no_connect + MPN emission. Skill review now: 1 error (SS-001
sourcing gate, needs passive MPNs) + benign info; netlist connectivity intact.

Co-Authored-By: Claude Opus 4.8 <noreply@anthropic.com>
Parts:
- U10: MPN (none) -> TXS0108EPWR
Changed lines of the file:
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@@
 		(property "Footprint" "" (at 149.86 110.49 0)
+			(effects (font (size 1.27 1.27)) (hide yes)))
+		(property "MPN" "TXS0108EPWR" (at 149.86 110.49 0)
 			(effects (font (size 1.27 1.27)) (hide yes)))
 		(pin "1")
@@
 		(instances
 			(project "hardfuzz_v1"
-				(path "/d4330dca-89ae-4793-b016-d6c0afd5f7c5/834323ff-b24e-4edf-88f5-7fa6c7e5c4d6" (reference "U10") (unit 1))))
+				(path "/2a7cfa2e-8c6d-45dc-afe3-6b5c0cf25bc7/0e7f8766-b4f4-4bfe-8704-205b43950dd3" (reference "U10") (unit 1))))
 	)
 	(wire (pts (xy 139.70 102.87) (xy 137.16 102.87))
@@
 		(instances
 			(project "hardfuzz_v1"
-				(path "/d4330dca-89ae-4793-b016-d6c0afd5f7c5/834323ff-b24e-4edf-88f5-7fa6c7e5c4d6" (reference "#PWR20") (unit 1))))
+				(path "/2a7cfa2e-8c6d-45dc-afe3-6b5c0cf25bc7/0e7f8766-b4f4-4bfe-8704-205b43950dd3" (reference "#PWR20") (unit 1))))
 	)
 	(wire (pts (xy 129.54 59.69) (xy 129.54 62.23))
@@
 		(instances
 			(project "hardfuzz_v1"
-				(path "/d4330dca-89ae-4793-b016-d6c0afd5f7c5/834323ff-b24e-4edf-88f5-7fa6c7e5c4d6" (reference "#PWR21") (unit 1))))
+				(path "/2a7cfa2e-8c6d-45dc-afe3-6b5c0cf25bc7/0e7f8766-b4f4-4bfe-8704-205b43950dd3" (reference "#PWR21") (unit 1))))
 	)
 	(wire (pts (xy 149.86 154.94) (xy 149.86 152.40))
@@
 		(instances
 			(project "hardfuzz_v1"
-				(path "/d4330dca-89ae-4793-b016-d6c0afd5f7c5/834323ff-b24e-4edf-88f5-7fa6c7e5c4d6" (reference "C30") (unit 1))))
+				(path "/2a7cfa2e-8c6d-45dc-afe3-6b5c0cf25bc7/0e7f8766-b4f4-4bfe-8704-205b43950dd3" (reference "C30") (unit 1))))
 	)
 	(wire (pts (xy 110.49 96.52) (xy 110.49 93.98))
@@
 		(instances
 			(project "hardfuzz_v1"
-				(path "/d4330dca-89ae-4793-b016-d6c0afd5f7c5/834323ff-b24e-4edf-88f5-7fa6c7e5c4d6" (reference "C31") (unit 1))))
+				(path "/2a7cfa2e-8c6d-45dc-afe3-6b5c0cf25bc7/0e7f8766-b4f4-4bfe-8704-205b43950dd3" (reference "C31") (unit 1))))
 	)
 	(wire (pts (xy 190.50 96.52) (xy 190.50 93.98))
@@
 		(instances
 			(project "hardfuzz_v1"
-				(path "/d4330dca-89ae-4793-b016-d6c0afd5f7c5/834323ff-b24e-4edf-88f5-7fa6c7e5c4d6" (reference "R30") (unit 1))))
+				(path "/2a7cfa2e-8c6d-45dc-afe3-6b5c0cf25bc7/0e7f8766-b4f4-4bfe-8704-205b43950dd3" (reference "R30") (unit 1))))
 	)
 	(wire (pts (xy 129.54 71.12) (xy 129.54 68.58))
@@
 		(instances
 			(project "hardfuzz_v1"
-				(path "/d4330dca-89ae-4793-b016-d6c0afd5f7c5/834323ff-b24e-4edf-88f5-7fa6c7e5c4d6" (reference "R31") (unit 1))))
+				(path "/2a7cfa2e-8c6d-45dc-afe3-6b5c0cf25bc7/0e7f8766-b4f4-4bfe-8704-205b43950dd3" (reference "R31") (unit 1))))
 	)
 	(wire (pts (xy 209.55 76.20) (xy 209.55 73.66))
@@
 		(instances
 			(project "hardfuzz_v1"
-				(path "/d4330dca-89ae-4793-b016-d6c0afd5f7c5/834323ff-b24e-4edf-88f5-7fa6c7e5c4d6" (reference "R32") (unit 1))))
+				(path "/2a7cfa2e-8c6d-45dc-afe3-6b5c0cf25bc7/0e7f8766-b4f4-4bfe-8704-205b43950dd3" (reference "R32") (unit 1))))
 	)
 	(wire (pts (xy 222.25 76.20) (xy 222.25 73.66))
@@
 		(instances
 			(project "hardfuzz_v1"
-				(path "/d4330dca-89ae-4793-b016-d6c0afd5f7c5/834323ff-b24e-4edf-88f5-7fa6c7e5c4d6" (reference "R33") (unit 1))))
+				(path "/2a7cfa2e-8c6d-45dc-afe3-6b5c0cf25bc7/0e7f8766-b4f4-4bfe-8704-205b43950dd3" (reference "R33") (unit 1))))
 	)
 	(wire (pts (xy 250.19 66.04) (xy 250.19 63.50))
@@
 		(instances
 			(project "hardfuzz_v1"
-				(path "/d4330dca-89ae-4793-b016-d6c0afd5f7c5/834323ff-b24e-4edf-88f5-7fa6c7e5c4d6" (reference "R34") (unit 1))))
+				(path "/2a7cfa2e-8c6d-45dc-afe3-6b5c0cf25bc7/0e7f8766-b4f4-4bfe-8704-205b43950dd3" (reference "R34") (unit 1))))
 	)
 	(wire (pts (xy 250.19 91.44) (xy 250.19 88.90))
@@
 		(instances
 			(project "hardfuzz_v1"
-				(path "/d4330dca-89ae-4793-b016-d6c0afd5f7c5/834323ff-b24e-4edf-88f5-7fa6c7e5c4d6" (reference "C32") (unit 1))))
+				(path "/2a7cfa2e-8c6d-45dc-afe3-6b5c0cf25bc7/0e7f8766-b4f4-4bfe-8704-205b43950dd3" (reference "C32") (unit 1))))
 	)
 	(wire (pts (xy 267.97 78.74) (xy 267.97 76.20))
@@
 		(instances
 			(project "hardfuzz_v1"
-				(path "/d4330dca-89ae-4793-b016-d6c0afd5f7c5/834323ff-b24e-4edf-88f5-7fa6c7e5c4d6" (reference "D20") (unit 1))))
+				(path "/2a7cfa2e-8c6d-45dc-afe3-6b5c0cf25bc7/0e7f8766-b4f4-4bfe-8704-205b43950dd3" (reference "D20") (unit 1))))
 	)
 	(wire (pts (xy 278.13 82.55) (xy 275.59 82.55))
@@
 		(instances
 			(project "hardfuzz_v1"
-				(path "/d4330dca-89ae-4793-b016-d6c0afd5f7c5/834323ff-b24e-4edf-88f5-7fa6c7e5c4d6" (reference "#PWR22") (unit 1))))
+				(path "/2a7cfa2e-8c6d-45dc-afe3-6b5c0cf25bc7/0e7f8766-b4f4-4bfe-8704-205b43950dd3" (reference "#PWR22") (unit 1))))
 	)
 	(wire (pts (xy 265.43 107.95) (xy 265.43 105.41))
@@
 		(instances
 			(project "hardfuzz_v1"
-				(path "/d4330dca-89ae-4793-b016-d6c0afd5f7c5/834323ff-b24e-4edf-88f5-7fa6c7e5c4d6" (reference "J2") (unit 1))))
+				(path "/2a7cfa2e-8c6d-45dc-afe3-6b5c0cf25bc7/0e7f8766-b4f4-4bfe-8704-205b43950dd3" (reference "J2") (unit 1))))
 	)
 	(wire (pts (xy 314.96 67.31) (xy 312.42 67.31))
@@
 		(instances
 			(project "hardfuzz_v1"
-				(path "/d4330dca-89ae-4793-b016-d6c0afd5f7c5/834323ff-b24e-4edf-88f5-7fa6c7e5c4d6" (reference "J3") (unit 1))))
+				(path "/2a7cfa2e-8c6d-45dc-afe3-6b5c0cf25bc7/0e7f8766-b4f4-4bfe-8704-205b43950dd3" (reference "J3") (unit 1))))
 	)
 	(wire (pts (xy 354.33 119.38) (xy 351.79 119.38))
@@
 		(instances
 			(project "hardfuzz_v1"
-				(path "/d4330dca-89ae-4793-b016-d6c0afd5f7c5/834323ff-b24e-4edf-88f5-7fa6c7e5c4d6" (reference "J4") (unit 1))))
+				(path "/2a7cfa2e-8c6d-45dc-afe3-6b5c0cf25bc7/0e7f8766-b4f4-4bfe-8704-205b43950dd3" (reference "J4") (unit 1))))
 	)
 	(wire (pts (xy 415.29 124.46) (xy 412.75 124.46))
@@
 )
 	(sheet_instances
-		(path "/834323ff-b24e-4edf-88f5-7fa6c7e5c4d6" (page "5")))
+		(path "/0e7f8766-b4f4-4bfe-8704-205b43950dd3" (page "5")))
 	(embedded_fonts no)
 )

Commit message: hardware: generate placed PCB (hardfuzz_v1.kicad_pcb) + footprints; rename root
kigen_pcb.py generates the PCB from the schematic netlist: loads each part's
stock .kicad_mod, shelf-packs footprints (origin-offset so courtyards don't
overlap), injects pad nets, and adds a board outline + 2-layer stackup. Loads in
pcbnew with 68 footprints and 302 nets on the right pads; the 317 'unconnected'
are the unrouted nets (routing is interactive/autorouter — the generator sets it
up, doesn't draw copper).

Also: assigned real footprints to the 6 ICs that lacked them and fixed 2 wrong
names (all now resolve, incl BGA-324 + QFN-64). Renamed the root schematic/PCB to
hardfuzz_v1.* so the project opens linked as hardfuzz_v1.kicad_pro.

Co-Authored-By: Claude Opus 4.8 <noreply@anthropic.com>
Parts:
- U10: footprint (none) -> Package_SO:TSSOP-20_4.4x6.5mm_P0.65mm
Changed lines of the file:
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@@
 		(property "Value" "TXS0108EPW" (at 73.71 80.07 0)
 			(effects (font (size 1.27 1.27)) (justify left)))
-		(property "Footprint" "" (at 71.17 78.80 0)
+		(property "Footprint" "Package_SO:TSSOP-20_4.4x6.5mm_P0.65mm" (at 71.17 78.80 0)
 			(effects (font (size 1.27 1.27)) (hide yes)))
 		(property "MPN" "TXS0108EPWR" (at 71.17 78.80 0)
@@
 		(instances
 			(project "hardfuzz_v1"
-				(path "/ba6f588c-ef80-4b6d-a64b-de96b4dacc26/9c141e12-a5e2-408d-b2ef-7a163e866b59" (reference "U10") (unit 1))))
+				(path "/287a9ed2-a26a-4469-8d2c-da808579c5eb/0e10d402-24c3-47d1-9160-0ec9ff65fe17" (reference "U10") (unit 1))))
 	)
 	(wire (pts (xy 61.01 71.18) (xy 58.47 71.18))
@@
 		(instances
 			(project "hardfuzz_v1"
-				(path "/ba6f588c-ef80-4b6d-a64b-de96b4dacc26/9c141e12-a5e2-408d-b2ef-7a163e866b59" (reference "#PWR20") (unit 1))))
+				(path "/287a9ed2-a26a-4469-8d2c-da808579c5eb/0e10d402-24c3-47d1-9160-0ec9ff65fe17" (reference "#PWR20") (unit 1))))
 	)
 	(wire (pts (xy 50.85 28.00) (xy 50.85 30.54))
@@
 		(instances
 			(project "hardfuzz_v1"
-				(path "/ba6f588c-ef80-4b6d-a64b-de96b4dacc26/9c141e12-a5e2-408d-b2ef-7a163e866b59" (reference "#PWR21") (unit 1))))
+				(path "/287a9ed2-a26a-4469-8d2c-da808579c5eb/0e10d402-24c3-47d1-9160-0ec9ff65fe17" (reference "#PWR21") (unit 1))))
 	)
 	(wire (pts (xy 71.17 123.25) (xy 71.17 120.71))
@@
 		(instances
 			(project "hardfuzz_v1"
-				(path "/ba6f588c-ef80-4b6d-a64b-de96b4dacc26/9c141e12-a5e2-408d-b2ef-7a163e866b59" (reference "C30") (unit 1))))
+				(path "/287a9ed2-a26a-4469-8d2c-da808579c5eb/0e10d402-24c3-47d1-9160-0ec9ff65fe17" (reference "C30") (unit 1))))
 	)
 	(wire (pts (xy 31.80 64.83) (xy 31.80 62.29))
@@
 		(instances
 			(project "hardfuzz_v1"
-				(path "/ba6f588c-ef80-4b6d-a64b-de96b4dacc26/9c141e12-a5e2-408d-b2ef-7a163e866b59" (reference "C31") (unit 1))))
+				(path "/287a9ed2-a26a-4469-8d2c-da808579c5eb/0e10d402-24c3-47d1-9160-0ec9ff65fe17" (reference "C31") (unit 1))))
 	)
 	(wire (pts (xy 111.81 64.83) (xy 111.81 62.29))
@@
 		(instances
 			(project "hardfuzz_v1"
-				(path "/ba6f588c-ef80-4b6d-a64b-de96b4dacc26/9c141e12-a5e2-408d-b2ef-7a163e866b59" (reference "R30") (unit 1))))
+				(path "/287a9ed2-a26a-4469-8d2c-da808579c5eb/0e10d402-24c3-47d1-9160-0ec9ff65fe17" (reference "R30") (unit 1))))
 	)
 	(wire (pts (xy 50.85 39.43) (xy 50.85 36.89))
@@
 		(instances
 			(project "hardfuzz_v1"
-				(path "/ba6f588c-ef80-4b6d-a64b-de96b4dacc26/9c141e12-a5e2-408d-b2ef-7a163e866b59" (reference "R31") (unit 1))))
+				(path "/287a9ed2-a26a-4469-8d2c-da808579c5eb/0e10d402-24c3-47d1-9160-0ec9ff65fe17" (reference "R31") (unit 1))))
 	)
 	(wire (pts (xy 130.86 44.51) (xy 130.86 41.97))
@@
 		(instances
 			(project "hardfuzz_v1"
-				(path "/ba6f588c-ef80-4b6d-a64b-de96b4dacc26/9c141e12-a5e2-408d-b2ef-7a163e866b59" (reference "R32") (unit 1))))
+				(path "/287a9ed2-a26a-4469-8d2c-da808579c5eb/0e10d402-24c3-47d1-9160-0ec9ff65fe17" (reference "R32") (unit 1))))
 	)
 	(wire (pts (xy 143.56 44.51) (xy 143.56 41.97))
@@
 		(instances
 			(project "hardfuzz_v1"
-				(path "/ba6f588c-ef80-4b6d-a64b-de96b4dacc26/9c141e12-a5e2-408d-b2ef-7a163e866b59" (reference "R33") (unit 1))))
+				(path "/287a9ed2-a26a-4469-8d2c-da808579c5eb/0e10d402-24c3-47d1-9160-0ec9ff65fe17" (reference "R33") (unit 1))))
 	)
 	(wire (pts (xy 171.50 34.35) (xy 171.50 31.81))
@@
 		(instances
 			(project "hardfuzz_v1"
-				(path "/ba6f588c-ef80-4b6d-a64b-de96b4dacc26/9c141e12-a5e2-408d-b2ef-7a163e866b59" (reference "R34") (unit 1))))
+				(path "/287a9ed2-a26a-4469-8d2c-da808579c5eb/0e10d402-24c3-47d1-9160-0ec9ff65fe17" (reference "R34") (unit 1))))
 	)
 	(wire (pts (xy 171.50 59.75) (xy 171.50 57.21))
@@
 		(instances
 			(project "hardfuzz_v1"
-				(path "/ba6f588c-ef80-4b6d-a64b-de96b4dacc26/9c141e12-a5e2-408d-b2ef-7a163e866b59" (reference "C32") (unit 1))))
+				(path "/287a9ed2-a26a-4469-8d2c-da808579c5eb/0e10d402-24c3-47d1-9160-0ec9ff65fe17" (reference "C32") (unit 1))))
 	)
 	(wire (pts (xy 189.28 47.05) (xy 189.28 44.51))
@@
 		(instances
 			(project "hardfuzz_v1"
-				(path "/ba6f588c-ef80-4b6d-a64b-de96b4dacc26/9c141e12-a5e2-408d-b2ef-7a163e866b59" (reference "D20") (unit 1))))
+				(path "/287a9ed2-a26a-4469-8d2c-da808579c5eb/0e10d402-24c3-47d1-9160-0ec9ff65fe17" (reference "D20") (unit 1))))
 	)
 	(wire (pts (xy 199.44 50.86) (xy 196.90 50.86))
@@
 		(instances
 			(project "hardfuzz_v1"
-				(path "/ba6f588c-ef80-4b6d-a64b-de96b4dacc26/9c141e12-a5e2-408d-b2ef-7a163e866b59" (reference "#PWR22") (unit 1))))
+				(path "/287a9ed2-a26a-4469-8d2c-da808579c5eb/0e10d402-24c3-47d1-9160-0ec9ff65fe17" (reference "#PWR22") (unit 1))))
 	)
 	(wire (pts (xy 186.74 76.26) (xy 186.74 73.72))
@@
 		(instances
 			(project "hardfuzz_v1"
-				(path "/ba6f588c-ef80-4b6d-a64b-de96b4dacc26/9c141e12-a5e2-408d-b2ef-7a163e866b59" (reference "J2") (unit 1))))
+				(path "/287a9ed2-a26a-4469-8d2c-da808579c5eb/0e10d402-24c3-47d1-9160-0ec9ff65fe17" (reference "J2") (unit 1))))
 	)
 	(wire (pts (xy 236.27 35.62) (xy 233.73 35.62))
@@
 		(instances
 			(project "hardfuzz_v1"
-				(path "/ba6f588c-ef80-4b6d-a64b-de96b4dacc26/9c141e12-a5e2-408d-b2ef-7a163e866b59" (reference "J3") (unit 1))))
+				(path "/287a9ed2-a26a-4469-8d2c-da808579c5eb/0e10d402-24c3-47d1-9160-0ec9ff65fe17" (reference "J3") (unit 1))))
 	)
 	(wire (pts (xy 275.64 87.69) (xy 273.10 87.69))
@@
 		(instances
 			(project "hardfuzz_v1"
-				(path "/ba6f588c-ef80-4b6d-a64b-de96b4dacc26/9c141e12-a5e2-408d-b2ef-7a163e866b59" (reference "J4") (unit 1))))
+				(path "/287a9ed2-a26a-4469-8d2c-da808579c5eb/0e10d402-24c3-47d1-9160-0ec9ff65fe17" (reference "J4") (unit 1))))
 	)
 	(wire (pts (xy 336.60 92.77) (xy 334.06 92.77))
@@
 )
 	(sheet_instances
-		(path "/9c141e12-a5e2-408d-b2ef-7a163e866b59" (page "5")))
+		(path "/0e10d402-24c3-47d1-9160-0ec9ff65fe17" (page "5")))
 	(embedded_fonts no)
 )
